Commit message: update IK controller with QP

File: PythonRobotics/RoboticControl/ur5/ur5.urdf (robot description, URDF)
Before this commit: robot ur5, 7 links, 7 joints
Links:
- added link fake_pinch_link, mass 1e-3; collision cylinder length=0.6 radius=0.2; visual cylinder length=0.6 radius=0.2
Joints:
- added joint pinch_joint: type fixed, parent wrist_3_link, child fake_pinch_link, origin xyz=0 0.225 0 rpy=-1.5707963 0.0 0.0

Commit message: update ur5 model

File: PythonRobotics/RoboticControl/ur5/ur5.urdf (robot description, URDF)
Before this commit: robot ur5, 8 links, 8 joints
Joints:
- joint wrist_2_joint: origin xyz=0.0 0.093 0.0 rpy=0.0 0.0 0.0 -> xyz=0.0 0.127 0.0 rpy=0.0 0.0 0.0
- joint wrist_3_joint: origin xyz=0 0 0.09465 rpy=0.0 0.0 0.0 -> xyz=0 0 0.1 rpy=0.0 0.0 0.0
