Commit message: update

File: PythonRobotics/RobotSim/assets/urdf/anymal_b_simple_description/urdf/anymal.urdf (robot description, URDF)
Before this commit: robot anymal, 21 links, 20 joints
Links:
- link LF_ADAPTER: geometry collision cylinder length=0.32125 radius=0.015; visual mesh filename=/home/tyx/CodeBase/BEATPython/PythonRobotics/RobotSim/asset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 scale=0.001 0.001 0.001
- link LF_HIP: geometry collision cylinder length=0.03 radius=0.045; collision cylinder length=0.1 radius=0.08
- link LF_SHANK: geometry collision box size=0.08 0.07 0.13; visual mesh filename=/home/tyx/CodeBase/BEATPython/PythonRobotics/RobotSim/asset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 scale=0.001 0.001 0.001
- link LF_THIGH: geometry collision box size=0.08 0.04 0.25; collision cylinder length=0.12 radius=0.06
- link LH_ADAPTER: geometry collision cylinder length=0.32125 radius=0.015; visual mesh filename=/home/tyx/CodeBase/BEATPython/PythonRobotics/RobotSim/asset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 scale=0.001 0.001 0.001
- link LH_HIP: geometry collision cylinder length=0.03 radius=0.045; collision cylinder length=0.1 radius=0.08
- link LH_SHANK: geometry collision box size=0.08 0.07 0.13; visual mesh filename=/home/tyx/CodeBase/BEATPython/PythonRobotics/RobotSim/asset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 scale=0.001 0.001 0.001
- link LH_THIGH: geometry collision box size=0.08 0.04 0.25; collision cylinder length=0.12 radius=0.06
- link RF_ADAPTER: geometry collision cylinder length=0.32125 radius=0.015; visual mesh filename=/home/tyx/CodeBase/BEATPython/PythonRobotics/RobotSim/asset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 scale=0.001 0.001 0.001
- link RF_HIP: geometry collision cylinder length=0.03 radius=0.045; collision cylinder length=0.1 radius=0.08
- link RF_SHANK: geometry collision box size=0.08 0.07 0.13; visual mesh filename=/home/tyx/CodeBase/BEATPython/PythonRobotics/RobotSim/asset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 scale=0.001 0.001 0.001
- link RF_THIGH: geometry collision box size=0.08 0.04 0.25; collision cylinder length=0.12 radius=0.06
- link RH_ADAPTER: geometry collision cylinder length=0.32125 radius=0.015; visual mesh filename=/home/tyx/CodeBase/BEATPython/PythonRobotics/RobotSim/asset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 scale=0.001 0.001 0.001
- link RH_HIP: geometry collision cylinder length=0.03 radius=0.045; collision cylinder length=0.1 radius=0.08
- link RH_SHANK: geometry collision box size=0.08 0.07 0.13; visual mesh filename=/home/tyx/CodeBase/BEATPython/PythonRobotics/RobotSim/asset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 scale=0.001 0.001 0.001
- link RH_THIGH: geometry collision box size=0.08 0.04 0.25; collision cylinder length=0.12 radius=0.06
- link base: geometry collision box size=0.1 0.1 0.07; collision box size=0.1 0.1 0.07

File: PythonRobotics/RoboticControl/ur5/ur5.urdf (robot description, URDF)
Before this commit: robot ur5, 8 links, 8 joints
Links:
- link base_link: geometry collision mesh filename=ur5/collision/base.obj; visual mesh filename=ur5/assets/base.obj
- link forearm_link: geometry collision mesh filename=ur5/collision/forearm.obj; visual mesh filename=ur5/assets/forearm.obj
- link shoulder_link: geometry collision mesh filename=ur5/collision/shoulder.obj; visual mesh filename=ur5/assets/shoulder.obj
- link upper_arm_link: geometry collision mesh filename=ur5/collision/upperarm.obj; visual mesh filename=ur5/assets/upperarm.obj
- link wrist_1_link: geometry collision mesh filename=ur5/collision/wrist1.obj; visual mesh filename=ur5/assets/wrist1.obj
- link wrist_2_link: geometry collision mesh filename=ur5/collision/wrist2.obj; visual mesh filename=ur5/assets/wrist2.obj
- link wrist_3_link: geometry collision mesh filename=ur5/collision/wrist3.obj; visual mesh filename=ur5/assets/wrist3.obj
